Commit message: loading the compiles iris.sdf

File: models/iris/iris.sdf.xacro (robot description, xacro)
@@ -3,5 +3,6 @@
   <xacro:arg name='mavlink_tcp_port' default='4560' />
   <xacro:arg name='qgc_udp_port' default='4560' />
-  <xacro:arg name='enable_camera' default='true' />
+  <xacro:arg name='enable_camera' default='false' />
+  <xacro:arg name='enable_stereo_camera' default='true' />
   <xacro:arg name='camera_pose' default='0 0 0 0 0 0' />
   <xacro:arg name='camera_udp_port' default='5600' />
@@ -595,4 +596,19 @@
     </joint>
   </xacro:if>
+  <xacro:if value="$(arg enable_stereo_camera)">
+    <xacro:include filename="$(arg rotors_description_dir)/stereo_cam/stereo_cam.sdf.xacro">
+    </xacro:include>
+    <joint name="stereo_cam_joint" type="fixed">
+      <child>stereo_cam::link</child>
+      <parent>base_link</parent>
+      <axis>
+  <xyz>0 0 1</xyz>
+  <limit>
+    <upper>0</upper>
+    <lower>0</lower>
+  </limit>
+      </axis>
+    </joint>
+  </xacro:if>
   </model>
 </sdf>
